Commit message: URDF con fricción de orugas

File: urdf/ROBOT_ZUMO_URDF.SLDASM.urdf (robot description, URDF)
Before this commit: robot ROBOT_ZUMO_URDF.SLDASM, 8 links, 7 joints
Links:
- link left_track_link: mass None -> 0.001; geometry collision mesh filename=package://zumo_1/meshes/left_track_link.STL; visual mesh filename=package://zumo_1/meshes/left_track_link.STL
- link right_track_link: mass None -> 0.001; geometry collision mesh filename=package://zumo_1/meshes/right_track_link.STL; visual mesh filename=package://zumo_1/meshes/right_track_link.STL
Joints:
- joint left_track_joint: axis 0 0 0 -> (none)
- joint right_track_joint: axis 0 0 0 -> (none)
